File: kicad_files/pico.kicad_pcb (KiCad board)
At the start: 2 copper layers, 131.4 x 96.5 mm, 84 parts, among them K0 KEYSW, K1 KEYSW, K10 KEYSW, K11 KEYSW, K12 KEYSW, K13 KEYSW, K14 KEYSW, K15 KEYSW, K16 KEYSW, K2 KEYSW, K20 KEYSW, K21 KEYSW, K22 KEYSW, K23 KEYSW, K24 KEYSW, K25 KEYSW, K26 KEYSW, K3 KEYSW, K30 KEYSW, K31 KEYSW, K32 KEYSW, K33 KEYSW, K34 KEYSW, K35 KEYSW, K36 KEYSW, K4 KEYSW, K40 KEYSW, K41 KEYSW, K42 KEYSW, K43 KEYSW, K44 KEYSW, K45 KEYSW, K46 KEYSW, K5 KEYSW, K6 KEYSW, U1 ProMicro

Commit message: Modified README. (#4)
Parts:
- TRRS1: moved to B.Cu
- moved D3 1.00 mm to (138.5, 55.3)
- moved R2 1.00 mm to (138.5, 51.8)
- turned K0 to 270 degrees
- turned K1 to 270 degrees
- turned TRRS1 to 180 degrees
Routing:
- net Net-(D1-Pad2): track 18.9 -> 30.9 mm
- net Net-(D0-Pad2): track 24.2 -> 36.0 mm
- net col1: track 97.5 -> 106.0 mm
- net GND: track 226.9 -> 230.6 mm, vias 0 -> 1
- net SCL: track 71.9 -> 69.2 mm
- net row0: track 162.4 -> 164.9 mm
- net col0: track 103.4 -> 100.9 mm
- net SDA: track 72.8 -> 75.2 mm
- net VCC: track 212.1 -> 210.7 mm
- net col2: track 117.0 -> 116.1 mm
- net col4: track 140.4 -> 139.6 mm
Other:
- board text added: "Mounting"
- board text added: "Surface"
- board text removed: "Mounting Surface"
